Commit message: WIP chessbots

File: linorobot2_description/urdf/2wd_properties.urdf.xacro (robot description, xacro)
@@ -1,6 +1,6 @@
 <?xml version="1.0"?>
 <robot xmlns:xacro="http://ros.org/wiki/xacro">
-  <xacro:property name="base_length" value="0.24" />
-  <xacro:property name="base_width" value="0.275" />
+  <xacro:property name="base_length" value="0.15" />
+  <xacro:property name="base_width" value="0.15" />
   <xacro:property name="base_height" value="0.003" />
   <xacro:property name="base_mass" value="1" />
@@ -11,5 +11,5 @@
   <xacro:property name="wheel_width" value="0.01" />
   <xacro:property name="wheel_pos_x" value="0.0" />
-  <xacro:property name="wheel_pos_y" value="0.13" />
+  <xacro:property name="wheel_pos_y" value="0.08" />
   <xacro:property name="wheel_pos_z" value="-0.03" />
   <xacro:property name="wheel_mass" value=".1" />
@@ -21,8 +21,8 @@
   <!-- <xacro:property name="wheel_mesh_file" value="file://$(find linorobot2_description)/meshes/tire.dae" /> -->
   <xacro:property name="laser_pose">
-    <origin xyz="0.12 0 0.33" rpy="0 0 0"/>
+    <origin xyz="0 0 0.08" rpy="0 0 0"/>
   </xacro:property>
   <xacro:property name="depth_sensor_pose">
-    <origin xyz="0.14 0.0 0.045" rpy="0 0 0"/>
+    <origin xyz="0.07 0.0 0.025" rpy="0 0 0"/>
   </xacro:property>
 </robot>
