Commit message: Add USB camera support with TF integration
Add a UVC USB camera to bringup, gated on LINOROBOT2_USB_CAMERA:
- usb_cam driver publishes full-res /usb_camera/image_raw for local use
- image_proc resize node publishes a downscaled, JPEG-compressed stream
  (/usb_camera/downscaled/image_raw/compressed) for slow networks,
  toggleable via LINOROBOT2_USB_CAMERA_STREAM
- Add usb_camera_link + REP-103 usb_camera_optical_link to the URDF of all
  robot models, positioned per-robot via usb_camera_pose
- Driver stamps images with usb_camera_optical_link for correct projection
- Document setup, topics, and tuning in ROBOT_INSTALLATION.md

Also resolve a pre-existing robomow_612p delete/modify conflict (keeping the
files) and ignore build/install/log artifacts.

Co-Authored-By: Claude Opus 4.8 <noreply@anthropic.com>

File: linorobot2_description/urdf/2wd_properties.urdf.xacro (robot description, xacro)
@@ -26,3 +26,6 @@
     <origin xyz="0.14 0.0 0.045" rpy="0 0 0"/>
   </xacro:property>
+  <xacro:property name="usb_camera_pose">
+    <origin xyz="0.14 0.0 0.075" rpy="0 0 0"/>
+  </xacro:property>
 </robot>

File: linorobot2_description/urdf/4wd_properties.urdf.xacro (robot description, xacro)
@@ -24,3 +24,6 @@
     <origin xyz="-0.065 0 0.255" rpy="0 0 0"/>
   </xacro:property>
+  <xacro:property name="usb_camera_pose">
+    <origin xyz="-0.065 0 0.285" rpy="0 0 0"/>
+  </xacro:property>
 </robot>

File: linorobot2_description/urdf/mecanum_properties.urdf.xacro (robot description, xacro)
@@ -24,3 +24,6 @@
     <origin xyz="0.2375 0 0.06" rpy="0 0 0"/>
   </xacro:property>
+  <xacro:property name="usb_camera_pose">
+    <origin xyz="0.2375 0 0.09" rpy="0 0 0"/>
+  </xacro:property>
 </robot>

File: linorobot2_description/urdf/robots/2wd.urdf.xacro (robot description, xacro)
@@ -10,4 +10,5 @@
   <xacro:include filename="$(find linorobot2_description)/urdf/sensors/generic_laser.urdf.xacro" />
   <xacro:include filename="$(find linorobot2_description)/urdf/sensors/depth_sensor.urdf.xacro" />
+  <xacro:include filename="$(find linorobot2_description)/urdf/sensors/usb_camera.urdf.xacro" />
   <xacro:include filename="$(find linorobot2_description)/urdf/controllers/diff_drive.urdf.xacro" />
   <xacro:base
@@ -65,4 +66,7 @@
     <xacro:insert_block name="depth_sensor_pose" />
   </xacro:depth_sensor>
+  <xacro:usb_camera>
+    <xacro:insert_block name="usb_camera_pose" />
+  </xacro:usb_camera>
   <xacro:diff_drive_controller
     wheel_separation="${wheel_pos_y * 2}"

File: linorobot2_description/urdf/robots/mecanum.urdf.xacro (robot description, xacro)
@@ -8,4 +8,5 @@
   <xacro:include filename="$(find linorobot2_description)/urdf/sensors/generic_laser.urdf.xacro" />
   <xacro:include filename="$(find linorobot2_description)/urdf/sensors/depth_sensor.urdf.xacro" />
+  <xacro:include filename="$(find linorobot2_description)/urdf/sensors/usb_camera.urdf.xacro" />
   <xacro:include filename="$(find linorobot2_description)/urdf/controllers/omni_drive.urdf.xacro" />
   <xacro:base
@@ -65,4 +66,7 @@
     <xacro:insert_block name="depth_sensor_pose" />
   </xacro:depth_sensor>
+  <xacro:usb_camera>
+    <xacro:insert_block name="usb_camera_pose" />
+  </xacro:usb_camera>
   <xacro:omni_drive_controller
     wheel_separation="${wheel_pos_y * 2}"

File: linorobot2_description/urdf/robots/robomow_612p.urdf.xacro (robot description, xacro)
@@ -1,7 +1,9 @@
 <?xml version="1.0"?>
-<robot name="linorobot2_4wd" xmlns:xacro="http://ros.org/wiki/xacro">
-  <xacro:include filename="$(find linorobot2_description)/urdf/4wd_properties.urdf.xacro" />
+<robot name="robomow_612p" xmlns:xacro="http://ros.org/wiki/xacro">
+  <xacro:arg name="sim" default="false" />
+  <xacro:include filename="$(find linorobot2_description)/urdf/robomow_612p_properties.urdf.xacro" />
   <xacro:include filename="$(find linorobot2_description)/urdf/mech/base.urdf.xacro" />
   <xacro:include filename="$(find linorobot2_description)/urdf/mech/wheel.urdf.xacro" />
+  <xacro:include filename="$(find linorobot2_description)/urdf/mech/caster_wheel.urdf.xacro" />
   <xacro:include filename="$(find linorobot2_description)/urdf/sensors/plugins.urdf.xacro" />
   <xacro:include filename="$(find linorobot2_description)/urdf/sensors/imu.urdf.xacro" />
@@ -9,5 +11,5 @@
   <xacro:include filename="$(find linorobot2_description)/urdf/sensors/depth_sensor.urdf.xacro" />
   <xacro:include filename="$(find linorobot2_description)/urdf/sensors/usb_camera.urdf.xacro" />
-  <xacro:include filename="$(find linorobot2_description)/urdf/controllers/skid_steer.urdf.xacro" />
+  <xacro:include filename="$(find linorobot2_description)/urdf/controllers/diff_drive.urdf.xacro" />
   <xacro:base
     length="${base_length}"
@@ -20,5 +22,5 @@
   />
   <xacro:wheel
-    side="front_left"
+    side="left"
     radius="${wheel_radius}"
     width="${wheel_width}"
@@ -30,5 +32,5 @@
   />
   <xacro:wheel
-    side="front_right"
+    side="right"
     radius="${wheel_radius}"
     width="${wheel_width}"
@@ -39,24 +41,13 @@
     mesh_file="${wheel_mesh_file}"
   />
-  <xacro:wheel
-    side="rear_left"
-    radius="${wheel_radius}"
-    width="${wheel_width}"
-    pos_x="${-wheel_pos_x}"
-    pos_y="${wheel_pos_y}"
-    pos_z="${wheel_pos_z}"
-    mass="${wheel_mass}"
-    mesh_file="${wheel_mesh_file}"
-  />
-  <xacro:wheel
-    side="rear_right"
-    radius="${wheel_radius}"
-    width="${wheel_width}"
-    pos_x="${-wheel_pos_x}"
-    pos_y="${-wheel_pos_y}"
-    pos_z="${wheel_pos_z}"
-    mass="${wheel_mass}"
-    mesh_file="${wheel_mesh_file}"
-  />
+  <xacro:if value="${front_caster_wheel}">
+    <xacro:caster_wheel
+      side="front"
+      mass="0.1"
+      base_length="${caster_pos_x}"
+      wheel_radius="${wheel_radius}"
+      wheel_pos_z="${wheel_pos_z}"
+    />
+  </xacro:if>
   <xacro:imu/>
   <xacro:generic_laser>

File: linorobot2_description/urdf/robots/vattenkar.urdf.xacro (robot description, xacro)
@@ -26,4 +26,5 @@
   <xacro:include filename="$(find linorobot2_description)/urdf/sensors/generic_laser.urdf.xacro" />
   <xacro:include filename="$(find linorobot2_description)/urdf/sensors/depth_sensor.urdf.xacro" />
+  <xacro:include filename="$(find linorobot2_description)/urdf/sensors/usb_camera.urdf.xacro" />
   <xacro:include filename="$(find linorobot2_description)/urdf/controllers/diff_drive.urdf.xacro" />
   <xacro:property name="laser_pose">
@@ -35,4 +36,7 @@
   <xacro:property name="depth_sensor_pose">
     <origin xyz="0.194 0.0 0.185" rpy="0 0 0"/>
+  </xacro:property>
+  <xacro:property name="usb_camera_pose">
+    <origin xyz="0.194 0.0 0.215" rpy="0 0 0"/>
   </xacro:property>
   <xacro:base
@@ -93,4 +97,7 @@
     <xacro:insert_block name="depth_sensor_pose" />
   </xacro:depth_sensor>
+  <xacro:usb_camera>
+    <xacro:insert_block name="usb_camera_pose" />
+  </xacro:usb_camera>
   <xacro:diff_drive_controller
     wheel_separation="${wheel_pos_y * 2}"

Commit message: Confine USB camera to mowberry platform per review
Revert camera edits to standard 2wd/4wd/mecanum/vattenkar robots and
their properties files. Rename robomow_612p{,_properties}.urdf.xacro to
mowberry{,_properties}.urdf.xacro and keep the camera there only.

Co-Authored-By: Claude Opus 4.8 <noreply@anthropic.com>

File: linorobot2_description/urdf/2wd_properties.urdf.xacro (robot description, xacro)
@@ -26,6 +26,3 @@
     <origin xyz="0.14 0.0 0.045" rpy="0 0 0"/>
   </xacro:property>
-  <xacro:property name="usb_camera_pose">
-    <origin xyz="0.14 0.0 0.075" rpy="0 0 0"/>
-  </xacro:property>
 </robot>

File: linorobot2_description/urdf/4wd_properties.urdf.xacro (robot description, xacro)
@@ -24,6 +24,3 @@
     <origin xyz="-0.065 0 0.255" rpy="0 0 0"/>
   </xacro:property>
-  <xacro:property name="usb_camera_pose">
-    <origin xyz="-0.065 0 0.285" rpy="0 0 0"/>
-  </xacro:property>
 </robot>

File: linorobot2_description/urdf/mecanum_properties.urdf.xacro (robot description, xacro)
@@ -24,6 +24,3 @@
     <origin xyz="0.2375 0 0.06" rpy="0 0 0"/>
   </xacro:property>
-  <xacro:property name="usb_camera_pose">
-    <origin xyz="0.2375 0 0.09" rpy="0 0 0"/>
-  </xacro:property>
 </robot>

File: linorobot2_description/urdf/robots/2wd.urdf.xacro (robot description, xacro)
@@ -10,5 +10,4 @@
   <xacro:include filename="$(find linorobot2_description)/urdf/sensors/generic_laser.urdf.xacro" />
   <xacro:include filename="$(find linorobot2_description)/urdf/sensors/depth_sensor.urdf.xacro" />
-  <xacro:include filename="$(find linorobot2_description)/urdf/sensors/usb_camera.urdf.xacro" />
   <xacro:include filename="$(find linorobot2_description)/urdf/controllers/diff_drive.urdf.xacro" />
   <xacro:base
@@ -66,7 +65,4 @@
     <xacro:insert_block name="depth_sensor_pose" />
   </xacro:depth_sensor>
-  <xacro:usb_camera>
-    <xacro:insert_block name="usb_camera_pose" />
-  </xacro:usb_camera>
   <xacro:diff_drive_controller
     wheel_separation="${wheel_pos_y * 2}"

File: linorobot2_description/urdf/robots/4wd.urdf.xacro (robot description, xacro)
@@ -8,5 +8,4 @@
   <xacro:include filename="$(find linorobot2_description)/urdf/sensors/generic_laser.urdf.xacro" />
   <xacro:include filename="$(find linorobot2_description)/urdf/sensors/depth_sensor.urdf.xacro" />
-  <xacro:include filename="$(find linorobot2_description)/urdf/sensors/usb_camera.urdf.xacro" />
   <xacro:include filename="$(find linorobot2_description)/urdf/controllers/skid_steer.urdf.xacro" />
   <xacro:base
@@ -66,7 +65,4 @@
     <xacro:insert_block name="depth_sensor_pose" />
   </xacro:depth_sensor>
-  <xacro:usb_camera>
-    <xacro:insert_block name="usb_camera_pose" />
-  </xacro:usb_camera>
   <xacro:diff_drive_controller
     wheel_separation="${wheel_pos_y * 2}"

File: linorobot2_description/urdf/robots/mecanum.urdf.xacro (robot description, xacro)
@@ -8,5 +8,4 @@
   <xacro:include filename="$(find linorobot2_description)/urdf/sensors/generic_laser.urdf.xacro" />
   <xacro:include filename="$(find linorobot2_description)/urdf/sensors/depth_sensor.urdf.xacro" />
-  <xacro:include filename="$(find linorobot2_description)/urdf/sensors/usb_camera.urdf.xacro" />
   <xacro:include filename="$(find linorobot2_description)/urdf/controllers/omni_drive.urdf.xacro" />
   <xacro:base
@@ -66,7 +65,4 @@
     <xacro:insert_block name="depth_sensor_pose" />
   </xacro:depth_sensor>
-  <xacro:usb_camera>
-    <xacro:insert_block name="usb_camera_pose" />
-  </xacro:usb_camera>
   <xacro:omni_drive_controller
     wheel_separation="${wheel_pos_y * 2}"

File: linorobot2_description/urdf/robots/mowberry.urdf.xacro (robot description, xacro)
@@ -1,6 +1,6 @@
 <?xml version="1.0"?>
-<robot name="robomow_612p" xmlns:xacro="http://ros.org/wiki/xacro">
+<robot name="mowberry" xmlns:xacro="http://ros.org/wiki/xacro">
   <xacro:arg name="sim" default="false" />
-  <xacro:include filename="$(find linorobot2_description)/urdf/robomow_612p_properties.urdf.xacro" />
+  <xacro:include filename="$(find linorobot2_description)/urdf/mowberry_properties.urdf.xacro" />
   <xacro:include filename="$(find linorobot2_description)/urdf/mech/base.urdf.xacro" />
   <xacro:include filename="$(find linorobot2_description)/urdf/mech/wheel.urdf.xacro" />

File: linorobot2_description/urdf/robots/vattenkar.urdf.xacro (robot description, xacro)
@@ -26,5 +26,4 @@
   <xacro:include filename="$(find linorobot2_description)/urdf/sensors/generic_laser.urdf.xacro" />
   <xacro:include filename="$(find linorobot2_description)/urdf/sensors/depth_sensor.urdf.xacro" />
-  <xacro:include filename="$(find linorobot2_description)/urdf/sensors/usb_camera.urdf.xacro" />
   <xacro:include filename="$(find linorobot2_description)/urdf/controllers/diff_drive.urdf.xacro" />
   <xacro:property name="laser_pose">
@@ -36,7 +35,4 @@
   <xacro:property name="depth_sensor_pose">
     <origin xyz="0.194 0.0 0.185" rpy="0 0 0"/>
-  </xacro:property>
-  <xacro:property name="usb_camera_pose">
-    <origin xyz="0.194 0.0 0.215" rpy="0 0 0"/>
   </xacro:property>
   <xacro:base
@@ -97,7 +93,4 @@
     <xacro:insert_block name="depth_sensor_pose" />
   </xacro:depth_sensor>
-  <xacro:usb_camera>
-    <xacro:insert_block name="usb_camera_pose" />
-  </xacro:usb_camera>
   <xacro:diff_drive_controller
     wheel_separation="${wheel_pos_y * 2}"
