Commit message: true urdf model of mowberry

File: linorobot2_description/urdf/mowberry_properties.urdf.xacro (robot description, xacro)
@@ -3,27 +3,28 @@
   <!-- Robomow 612P Dimensions (converted from inches to meters) -->
   <!-- 1 inch = 0.0254 meters -->
-  <!-- Horizontal distance between centers of wheels - 22 inch = 0.5588 m -->
-  <xacro:property name="base_width" value="0.5588" />
   <!-- Driving wheel diameter 8.5 inch -> radius 4.25 inch = 0.10795 m -->
   <xacro:property name="wheel_radius" value="0.10795" />
   <xacro:property name="wheel_width" value="0.090" />
-  <!-- Caster wheel position 19 inch from driving axle = 0.4826 m -->
   <xacro:property name="wheel_pos_x" value="0.0" />
-  <xacro:property name="wheel_pos_y" value="0.2794" /> <!-- base_width / 2 -->
-  <xacro:property name="wheel_pos_z" value="-0.0508" />
-  <!-- Caster wheel diameter 3.5 inch -> radius 1.75 inch = 0.04445 m -->
-  <xacro:property name="caster_radius" value="0.04445" />
-  <xacro:property name="caster_pos_x" value="0.5334" />
+  <xacro:property name="wheel_pos_y" value="0.27" />
+  <xacro:property name="wheel_pos_z" value="0.05" />
+  <xacro:property name="wheel_mass" value="1.0" />
+  <xacro:property name="wheel_torque" value="20" />
+  <!-- Caster wheel diameter 3.5 inch -> radius 1.75 inch = 0.044 m -->
+  <xacro:property name="caster_radius" value="0.044" />
+  <xacro:property name="caster_pos_x" value="0.50" />
   <xacro:property name="caster_pos_y" value="0.0" />
-  <xacro:property name="caster_pos_z" value="0.0" />
+  <xacro:property name="caster_pos_z" value="-0.006" />
+  <xacro:property name="front_caster_wheel" value="true" />
+  <xacro:property name="rear_caster_wheel" value="false" />
   <!-- Base dimensions -->
-  <xacro:property name="base_length" value="0.737" />
+  <xacro:property name="base_length" value="0.69" />
+  <xacro:property name="base_width" value="0.645" />
   <xacro:property name="base_height" value="0.2667" />
+  <!-- Base is offset from drive axle by half its length minus a little bit of rear overhang -->
+  <xacro:property name="base_offset_x" value="${base_length/2 - 0.07}" />
   <xacro:property name="base_mass" value="20.0" />
   <xacro:property name="base_mesh_file" value="" />
-  <xacro:property name="wheel_mass" value="1.0" />
-  <xacro:property name="wheel_torque" value="20" />
-  <xacro:property name="front_caster_wheel" value="true" />
-  <xacro:property name="rear_caster_wheel" value="false" />
+  <!-- set empty on the wheel_mesh_file to use geometry instead of mesh -->
   <xacro:property name="wheel_mesh_file" value="" />
   <xacro:property name="laser_pose">
@@ -34,5 +35,5 @@
   </xacro:property>
   <xacro:property name="usb_camera_pose">
-    <origin xyz="0.3 0 0.15" rpy="0 0 0"/>
+    <origin xyz="0.5 0 0.30" rpy="0 0 0"/>
   </xacro:property>
 </robot>
