Commit message: add bno085 imu, ld19 lidar

File: linorobot2_description/urdf/minniebot_properties.urdf.xacro (robot description, xacro)
@@ -3,5 +3,5 @@
   <xacro:property name="base_length" value="0.14" />
   <xacro:property name="base_width" value="0.14" />
-  <xacro:property name="base_height" value="0.01" />
+  <xacro:property name="base_height" value="0.003" />
   <xacro:property name="base_mass" value="0.5" />
   <!-- set empty on the wheel_mesh_file to use geometry instead of mesh -->
@@ -12,5 +12,5 @@
   <xacro:property name="wheel_pos_x" value="0.02" />
   <xacro:property name="wheel_pos_y" value="0.08" />
-  <xacro:property name="wheel_pos_z" value="-0.03" />
+  <xacro:property name="wheel_pos_z" value="-0.011" />
   <xacro:property name="wheel_mass" value=".05" />
   <xacro:property name="wheel_torque" value="20" />
@@ -20,12 +20,9 @@
   <xacro:property name="wheel_mesh_file" value="" />
   <!-- <xacro:property name="wheel_mesh_file" value="file://$(find linorobot2_description)/meshes/tire.dae" /> -->
+  <xacro:property name="imu_pose">
+    <origin xyz="0.048 0.054 0.01" rpy="0 0 0"/>
+  </xacro:property>
   <xacro:property name="laser_pose">
-    <origin xyz="0.010 0 0.04" rpy="0 0 0"/>
-  </xacro:property>
-  <xacro:property name="depth_sensor_pose">
-    <origin xyz="0.04 0.0 -0.03" rpy="0 0 0"/>
-  </xacro:property>
-  <xacro:property name="sonar_pose">
-    <origin xyz="0.05 0 0" rpy="0 0 0"/>
+    <origin xyz="0.022 0 0.056" rpy="0 0 0"/>
   </xacro:property>
 </robot>

File: linorobot2_description/urdf/robots/minniebot.urdf.xacro (robot description, xacro)
@@ -2,11 +2,11 @@
 <robot name="linorobot2_2wd" xmlns:xacro="http://ros.org/wiki/xacro">
   <xacro:arg name="sim" default="false" />
-  <xacro:include filename="$(find linorobot2_description)/urdf/2wd_properties.urdf.xacro" />
+  <xacro:include filename="$(find linorobot2_description)/urdf/minniebot_properties.urdf.xacro" />
   <xacro:include filename="$(find linorobot2_description)/urdf/mech/base.urdf.xacro" />
   <xacro:include filename="$(find linorobot2_description)/urdf/mech/wheel.urdf.xacro" />
   <xacro:include filename="$(find linorobot2_description)/urdf/mech/caster_wheel.urdf.xacro" />
   <xacro:include filename="$(find linorobot2_description)/urdf/sensors/plugins.urdf.xacro" />
-  <xacro:include filename="$(find linorobot2_description)/urdf/sensors/imu.urdf.xacro" />
-  <xacro:include filename="$(find linorobot2_description)/urdf/sensors/generic_laser.urdf.xacro" />
+  <xacro:include filename="$(find linorobot2_description)/urdf/sensors/bno085_imu.urdf.xacro" />
+  <xacro:include filename="$(find linorobot2_description)/urdf/sensors/ld19_laser_params.urdf.xacro" />
   <xacro:include filename="$(find linorobot2_description)/urdf/sensors/depth_sensor.urdf.xacro" />
   <xacro:include filename="$(find linorobot2_description)/urdf/controllers/diff_drive.urdf.xacro" />
@@ -58,11 +58,10 @@
     />
   </xacro:if>
-  <xacro:imu/>
-  <xacro:generic_laser>
+  <xacro:bno085_imu parent="base_link">
+    <xacro:insert_block name="imu_pose" />
+  </xacro:bno085_imu>
+  <xacro:ld19_laser_params>
     <xacro:insert_block name="laser_pose" />
-  </xacro:generic_laser>
-  <xacro:depth_sensor>
-    <xacro:insert_block name="depth_sensor_pose" />
-  </xacro:depth_sensor>
+  </xacro:ld19_laser_params>
   <xacro:diff_drive_controller
     wheel_separation="${wheel_pos_y * 2}"
